File: SnowMaker_RelayBoard/SMR.brd (EAGLE design)
At the start: 320 x 108.2 mm, 75 parts, among them CON1 CON-HARTING-26V

Commit message: temp1
Parts:
- removed XT10, XT11, XT12, XT13, XT14, XT15, XT16, XT17, XT18, XT19, XT20, XT21, XT22, XT23, XT24, XT25, XT4, XT5, XT6, XT7, XT8, XT9: FFKDS/V1-5.08-2, SHMT:FFKDS/V1-5.08-2
- U$1: device EN001_prj:EN001_OUTLINE -> SMR:108.2-OUTLINE
- XT1, XT2: value FFKDS/V1-5.08-2 -> FFKDS/V1-5.08-24; device SHMT:FFKDS/V1-5.08-2 -> SHMT:FFKDS/V1-5.08-24
- moved XT2 131.2 mm to (144.8, 104.1), turned to 180 degrees
- moved D19 117.2 mm to (63.5, 63.5), turned to 270 degrees
- moved D11 114.3 mm to (149.9, 26.7), turned to 90 degrees
- moved D7 114.3 mm to (106.7, 26.7), turned to 90 degrees
- moved D22 105.1 mm to (41.9, 63.5), turned to 270 degrees
- moved D12 105.0 mm to (149.9, 44.5), turned to 90 degrees
- moved D5 104.3 mm to (85.1, 26.7), turned to 90 degrees
- moved D9 104.1 mm to (128.3, 26.7), turned to 90 degrees
- moved D21 103.6 mm to (41.9, 81.3), turned to 270 degrees
- moved D24 102.4 mm to (20.3, 63.5), turned to 270 degrees
- moved D23 100.4 mm to (20.3, 81.3), turned to 270 degrees
- moved D18 97.9 mm to (85.1, 63.5), turned to 270 degrees
- moved D20 96.3 mm to (63.5, 81.3), turned to 270 degrees
- moved D16 95.2 mm to (106.7, 63.5), turned to 270 degrees
- moved D8 92.9 mm to (106.7, 44.5), turned to 90 degrees
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Connections:
- removed net N$49: KA1.4, XT1.2@1, XT1.2@2
- removed net N$50: KA1.5, XT1.1@1, XT1.1@2
- removed net N$61: KA3.5, XT3.1@1, XT3.1@2
- removed net N$62: KA3.4, XT3.2@1, XT3.2@2
- new net N$1: KA1.4, XT1.1@2, XT1.2@2
- new net N$2: KA1.5, XT1.1@1, XT1.2@1
- new net N$3: KA3.4, XT1.1@6, XT1.2@6
- new net N$4: KA3.5, XT1.1@5, XT1.2@5
- net +24V: now also XT3.2@1, XT3.2@2; no longer XT25.2@1, XT25.2@2
- net GND1: now also XT3.1@1, XT3.1@2; no longer XT25.1@1, XT25.1@2
- net N$100: now also XT1.1@24, XT1.2@24; no longer XT12.2@1, XT12.2@2
- net N$101: now also XT1.1@21, XT1.2@21; no longer XT11.1@1, XT11.1@2
- net N$102: now also XT1.1@22, XT1.2@22; no longer XT11.2@1, XT11.2@2
- net N$103: now also XT1.1@19, XT1.2@19; no longer XT10.1@1, XT10.1@2
- net N$104: now also XT1.1@20, XT1.2@20; no longer XT10.2@1, XT10.2@2
- net N$129: now also XT2.1@10, XT2.2@10; no longer XT17.2@1, XT17.2@2
- net N$130: now also XT2.1@9, XT2.2@9; no longer XT17.1@1, XT17.1@2
- net N$131: now also XT2.1@23, XT2.2@23; no longer XT24.1@1, XT24.1@2
- net N$132: now also XT2.1@24, XT2.2@24; no longer XT24.2@1, XT24.2@2
- net N$133: now also XT2.1@21, XT2.2@21; no longer XT23.1@1, XT23.1@2
- net N$134: now also XT2.1@22, XT2.2@22; no longer XT23.2@1, XT23.2@2
- net N$135: now also XT2.1@19, XT2.2@19; no longer XT22.1@1, XT22.1@2
- net N$136: now also XT2.1@20, XT2.2@20; no longer XT22.2@1, XT22.2@2
- net N$137: now also XT2.1@17, XT2.2@17; no longer XT21.1@1, XT21.1@2
- net N$138: now also XT2.1@18, XT2.2@18; no longer XT21.2@1, XT21.2@2
- net N$139: now also XT2.1@15, XT2.2@15; no longer XT20.1@1, XT20.1@2
- net N$140: now also XT2.1@16, XT2.2@16; no longer XT20.2@1, XT20.2@2
- net N$141: now also XT2.1@13, XT2.2@13; no longer XT19.1@1, XT19.1@2
- net N$142: now also XT2.1@14, XT2.2@14; no longer XT19.2@1, XT19.2@2
- net N$143: now also XT2.1@11, XT2.2@11; no longer XT18.1@1, XT18.1@2
- net N$144: now also XT2.1@12, XT2.2@12; no longer XT18.2@1, XT18.2@2
- net N$51: now also XT1.1@15, XT1.2@15; no longer XT8.1@1, XT8.1@2
- net N$52: now also XT1.1@16, XT1.2@16; no longer XT8.2@1, XT8.2@2
- net N$53: now also XT1.1@13, XT1.2@13; no longer XT7.1@1, XT7.1@2
- net N$54: now also XT1.1@14, XT1.2@14; no longer XT7.2@1, XT7.2@2
- net N$55: now also XT1.1@11, XT1.2@11; no longer XT6.1@1, XT6.1@2
- net N$56: now also XT1.1@12, XT1.2@12; no longer XT6.2@1, XT6.2@2
- net N$57: now also XT1.1@9, XT1.2@9; no longer XT5.1@1, XT5.1@2
- net N$58: now also XT1.1@10, XT1.2@10; no longer XT5.2@1, XT5.2@2
- net N$59: now also XT1.1@7, XT1.2@7; no longer XT4.1@1, XT4.1@2
- net N$60: now also XT1.1@8, XT1.2@8; no longer XT4.2@1, XT4.2@2
- net N$63: now also XT1.1@3, XT1.2@3; no longer XT2.1@1, XT2.1@2
- net N$64: now also XT1.1@4, XT1.2@4; no longer XT2.2@1, XT2.2@2
- net N$89: now also XT1.1@18, XT1.2@18; no longer XT9.2@1, XT9.2@2
- net N$90: now also XT1.1@17, XT1.2@17; no longer XT9.1@1, XT9.1@2
- net N$91: now also XT2.1@7, XT2.2@7; no longer XT16.1@1, XT16.1@2
- net N$92: now also XT2.1@8, XT2.2@8; no longer XT16.2@1, XT16.2@2
- net N$93: now also XT2.1@5, XT2.2@5; no longer XT15.1@1, XT15.1@2
- net N$94: now also XT2.1@6, XT2.2@6; no longer XT15.2@1, XT15.2@2
- net N$95: now also XT2.1@3, XT2.2@3; no longer XT14.1@1, XT14.1@2
- net N$96: now also XT2.1@4, XT2.2@4; no longer XT14.2@1, XT14.2@2
- net N$97: now also XT2.1@1, XT2.2@1; no longer XT13.1@1, XT13.1@2
- net N$98: now also XT2.1@2, XT2.2@2; no longer XT13.2@1, XT13.2@2
- net N$99: now also XT1.1@23, XT1.2@23; no longer XT12.1@1, XT12.1@2
Routing:
- net +24V: track 0.00 -> 862.9 mm
- net KA11: track 0.00 -> 153.9 mm, vias 0 -> 1
- net KA12: track 0.00 -> 144.1 mm
- net KA13: track 0.00 -> 135.0 mm
- net KA9: track 0.00 -> 130.2 mm, vias 0 -> 1
- net KA14: track 0.00 -> 127.4 mm, vias 0 -> 1
- net KA10: track 0.00 -> 121.5 mm
- net KA15: track 0.00 -> 112.4 mm
- net KA7: track 0.00 -> 106.5 mm, vias 0 -> 1
- net KA16: track 0.00 -> 106.3 mm, vias 0 -> 1
- net KA8: track 0.00 -> 100.1 mm
- net KA17: track 0.00 -> 88.6 mm
- net KA18: track 0.00 -> 85.8 mm, vias 0 -> 1
- net KA5: track 0.00 -> 82.8 mm, vias 0 -> 1
- net KA6: track 0.00 -> 79.0 mm
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Other:
- board size 320 x 108.2 mm -> 155 x 108.2 mm

Commit message: SMRB complete
Parts:
- added LOGO1: SY-LOGO_BOTTOM, LOGO:SY-LOGO_BOTTOM
- moved D19 17.8 mm to (63.5, 81.3)
- moved D20 17.8 mm to (63.5, 63.5)
- moved KA19 17.8 mm to (68.6, 81.3)
- moved KA20 17.8 mm to (68.6, 63.5)
Routing:
- net +24V: track 862.9 -> 913.2 mm
- net N$141: track 40.3 -> 20.4 mm
- net N$140: track 25.0 -> 43.0 mm
- net N$142: track 44.8 -> 27.1 mm
- net N$139: track 19.4 -> 37.1 mm
- net KA24: track 26.0 -> 23.9 mm
- net KA15: track 112.4 -> 110.7 mm
- net KA17: track 88.6 -> 87.2 mm
- net KA7: track 106.5 -> 107.7 mm
- net KA19: track 62.6 -> 63.6 mm, vias 1 -> 0
- net KA23: track 17.6 -> 16.6 mm
- net KA3: track 59.6 -> 60.6 mm
- net KA20: track 66.3 -> 65.4 mm, vias 0 -> 1
- net KA1: track 36.6 -> 37.4 mm
- net KA21: track 40.9 -> 40.0 mm
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Other:
- board text added: "0V"
- board text added: "0V 24V"
- board text added: "10C"
- board text added: "10NO"
- board text added: "11C"
- board text added: "11NO"
- board text added: "12C"
- board text added: "12NO"
- board text added: "13C"
- board text added: "13NO"
- board text added: "14C"
- board text added: "14NO"
- board text added: "15C"
- board text added: "15NO"
- board text added: "16C"
- board text added: "16NO"
- board text added: "17C"
- board text added: "17NO"
- board text added: "18C"
- board text added: "18NO"
- board text added: "19C"
- board text added: "19NO"
- board text added: "1C"
- board text added: "1NO"
- board text added: "2017/10/10"
- board text added: "20C"
- board text added: "20NO"
- board text added: "21C"
- board text added: "21NO"
- board text added: "22C"
- board text added: "22NO"
- board text added: "23C"
- board text added: "23NO"
- board text added: "24C"
- board text added: "24NO"
- board text added: "24V"
- board text added: "2C"
- board text added: "2NO"
- board text added: "3C"
- board text added: "3NO"
- board text added: "4C"
- board text added: "4NO"
- board text added: "5C"
- board text added: "5NO"
- board text added: "6C"
- board text added: "6NO"
- board text added: "7C"
- board text added: "7NO"
- board text added: "8C"
- board text added: "8NO"
- board text added: "9C"
- board text added: "9NO"
- board text added: "KA1"
- board text added: "KA2"
- board text added: "KA23"
- board text added: "KA24"
- board text added: "SMRB - V1"
