File: SnowMaker_RelayBoard/SMR.sch (EAGLE design)
At the start: 74 parts, among them CON1 CON-HARTING-26V

Commit message: temp1
Parts:
- removed XT10, XT11, XT12, XT13, XT14, XT15, XT16, XT17, XT18, XT19, XT20, XT21, XT22, XT23, XT24, XT25, XT4, XT5, XT6, XT7, XT8, XT9: FFKDS/V1-5.08-2, SHMT:FFKDS/V1-5.08-2
- XT1, XT2: value FFKDS/V1-5.08-2 -> FFKDS/V1-5.08-24; device SHMT:FFKDS/V1-5.08-2 -> SHMT:FFKDS/V1-5.08-24
Connections:
- removed net N$61: KA3G$2.NO, XT3-1.1
- removed net N$62: KA3G$2.COM, XT3-2.1
- new net N$3: KA3G$2.COM, XT1-6.1
- new net N$4: KA3G$2.NO, XT1-5.1
- net +24V: now also XT3-2.1; no longer XT25-2.1
- net GND1: now also XT3-1.1; no longer XT25-1.1
- net N$100: now also XT1-24.1; no longer XT12-2.1
- net N$101: now also XT1-21.1; no longer XT11-1.1
- net N$102: now also XT1-22.1; no longer XT11-2.1
- net N$103: now also XT1-19.1; no longer XT10-1.1
- net N$104: now also XT1-20.1; no longer XT10-2.1
- net N$129: now also XT2-10.1; no longer XT17-2.1
- net N$130: now also XT2-9.1; no longer XT17-1.1
- net N$131: now also XT2-23.1; no longer XT24-1.1
- net N$132: now also XT2-24.1; no longer XT24-2.1
- net N$133: now also XT2-21.1; no longer XT23-1.1
- net N$134: now also XT2-22.1; no longer XT23-2.1
- net N$135: now also XT2-19.1; no longer XT22-1.1
- net N$136: now also XT2-20.1; no longer XT22-2.1
- net N$137: now also XT2-17.1; no longer XT21-1.1
- net N$138: now also XT2-18.1; no longer XT21-2.1
- net N$139: now also XT2-15.1; no longer XT20-1.1
- net N$140: now also XT2-16.1; no longer XT20-2.1
- net N$141: now also XT2-13.1; no longer XT19-1.1
- net N$142: now also XT2-14.1; no longer XT19-2.1
- net N$143: now also XT2-11.1; no longer XT18-1.1
- net N$144: now also XT2-12.1; no longer XT18-2.1
- net N$51: now also XT1-15.1; no longer XT8-1.1
- net N$52: now also XT1-16.1; no longer XT8-2.1
- net N$53: now also XT1-13.1; no longer XT7-1.1
- net N$54: now also XT1-14.1; no longer XT7-2.1
- net N$55: now also XT1-11.1; no longer XT6-1.1
- net N$56: now also XT1-12.1; no longer XT6-2.1
- net N$57: now also XT1-9.1; no longer XT5-1.1
- net N$58: now also XT1-10.1; no longer XT5-2.1
- net N$59: now also XT1-7.1; no longer XT4-1.1
- net N$60: now also XT1-8.1; no longer XT4-2.1
- net N$63: now also XT1-3.1; no longer XT2-1.1
- net N$64: now also XT1-4.1; no longer XT2-2.1
- net N$89: now also XT1-18.1; no longer XT9-2.1
- net N$90: now also XT1-17.1; no longer XT9-1.1
- net N$91: now also XT2-7.1; no longer XT16-1.1
- net N$92: now also XT2-8.1; no longer XT16-2.1
- net N$93: now also XT2-5.1; no longer XT15-1.1
- net N$94: now also XT2-6.1; no longer XT15-2.1
- net N$95: now also XT2-3.1; no longer XT14-1.1
- net N$96: now also XT2-4.1; no longer XT14-2.1
- net N$97: now also XT2-1.1; no longer XT13-1.1
- net N$98: now also XT2-2.1; no longer XT13-2.1
- net N$99: now also XT1-23.1; no longer XT12-1.1
Other:
- moved on the sheet: XT2-1, XT2-2, XT3-1, XT3-2

Commit message: SMRB complete
Parts:
- added LOGO1: SY-LOGO_BOTTOM, LOGO:SY-LOGO_BOTTOM
Other:
- note added: "单独的继电器板，带24VDC端子 与主板通过牛角座相连，24V给光耦供电"
- note removed: "单独的继电器板，带24VDC端子 与主板通过牛角座相连，并送过去24V给光耦集"
- moved on the sheet: CON1, D1, D10, D11, D12, D13, D14, D15, D16, D17, D18, D19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
