File: snowmaker/SnowMaker_V1.0.brd (EAGLE design)
At the start: 315 x 108.2 mm, 571 parts, among them CON1 HR951180A, CON2 SWJ, IC1 ST3232BD, IC10 LM1117IDTX-3.3, IC11 SGM8584XS14, IC12 LM78M24, IC13 SGM8584XS14, IC14 SGM8584XS14, IC15 SGM8584XS14, IC2 ST3485EBD, IC3 W5500, IC4 SD2068, IC5 STM32F103VCT6, IC6 ULN2803, IC7 ULN2803, IC8 ULN2803, IC9 LM4040AIM3X-2.5, U1 LQ-BTM2540, X10 FFKDS/V1-5.08_MIDDLE, X11 FFKDS/V1-5.08_MIDDLE, X12 FFKDS/V1-5.08_MIDDLE, X13 FFKDS/V1-5.08_MIDDLE, X14 FFKDS/V1-5.08_MIDDLE, X15 FFKDS/V1-5.08_MIDDLE, X16 FFKDS/V1-5.08_MIDDLE, X17 FFKDS/V1-5.08_MIDDLE, X18 FFKDS/V1-5.08_MIDDLE, X19 FFKDS/V1-5.08_MIDDLE, X2 FFKDS/V1-5.08_FIRST, X20 FFKDS/V1-5.08_MIDDLE, X21 FFKDS/V1-5.08_MIDDLE, X22 FFKDS/V1-5.08_MIDDLE, X23 FFKDS/V1-5.08_MIDDLE, X24 FFKDS/V1-5.08_MIDDLE, X25 FFKDS/V1-5.08_MIDDLE, X26 FFKDS/V1-5.08_MIDDLE, X27 FFKDS/V1-5.08_MIDDLE, X28 FFKDS/V1-5.08_MIDDLE, X29 FFKDS/V1-5.08_MIDDLE, X3 FFKDS/V1-5.08_MIDDLE, X30 FFKDS/V1-5.08_MIDDLE, X31 FFKDS/V1-5.08_MIDDLE, X32 FFKDS/V1-5.08_MIDDLE, X33 FFKDS/V1-5.08_MIDDLE, X34 FFKDS/V1-5.08_MIDDLE, X35 FFKDS/V1-5.08_MIDDLE, X36 FFKDS/V1-5.08_MIDDLE, X37 FFKDS/V1-5.08_MIDDLE, X38 FFKDS/V1-5.08_MIDDLE, X39 FFKDS/V1-5.08_MIDDLE, X4 FFKDS/V1-5.08_MIDDLE, X40 FFKDS/V1-5.08_MIDDLE, X41 FFKDS/V1-5.08_LAST, X42 FFKDS/V1-5.08_MIDDLE, X43 FFKDS/V1-5.08_LAST, X44 FFKDS/V1-5.08_MIDDLE, X45 FFKDS/V1-5.08_MIDDLE, X46 FFKDS/V1-5.08_MIDDLE, X47 FFKDS/V1-5.08_MIDDLE, X48 FFKDS/V1-5.08_MIDDLE, X49 FFKDS/V1-5.08_MIDDLE, X5 FFKDS/V1-5.08_MIDDLE, X50 FFKDS/V1-5.08_MIDDLE, X51 FFKDS/V1-5.08_MIDDLE, X52 FFKDS/V1-5.08_MIDDLE, X53 FFKDS/V1-5.08_MIDDLE, X54 FFKDS/V1-5.08_MIDDLE, X55 FFKDS/V1-5.08_MIDDLE, X56 FFKDS/V1-5.08_MIDDLE, X57 FFKDS/V1-5.08_MIDDLE, X58 FFKDS/V1-5.08_FIRST, X59 FFKDS/V1-5.08_MIDDLE, X6 FFKDS/V1-5.08_MIDDLE, X60 FFKDS/V1-5.08_MIDDLE, X61 FFKDS/V1-5.08_MIDDLE, X62 FFKDS/V1-5.08_MIDDLE, X63 FFKDS/V1-5.08_MIDDLE, X64 FFKDS/V1-5.08_MIDDLE, X65 FFKDS/V1-5.08_MIDDLE, X66 FFKDS/V1-5.08_MIDDLE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

Commit message: PI fisrt commit
Parts:
- moved C59 13.2 mm to (303.3, 71.1), turned to 270 degrees
- moved EC1 2.30 mm to (290.6, 71.9)
- moved C16 2.29 mm to (264.1, 88.1)
- moved C18 2.29 mm to (259.0, 88.1)
- moved D1 2.29 mm to (270.5, 83.8)
- moved IC2 2.29 mm to (261.6, 83.5)
- moved L2 2.29 mm to (261.6, 87.3)
- moved R13 2.29 mm to (274.4, 83.8)
- moved R14 2.29 mm to (267.3, 85.2)
- moved R15 2.29 mm to (267.3, 82.2)
- moved R19 2.29 mm to (255.2, 83.5)
- moved R20 2.29 mm to (255.2, 81.6)
- moved R18 2.29 mm to (255.2, 85.5)
Connections:
- net N$61: now also X1.8
- net N$62: now also X1.6, X1.7; no longer X1.8
Routing:
- net +24V: track 274.8 -> 269.0 mm
- net N$62: track 35.8 -> 41.5 mm
- net N$36: track 18.0 -> 21.4 mm
- net N$35: track 19.2 -> 22.7 mm
- net N$41: track 17.8 -> 20.9 mm
- net N$42: track 21.6 -> 24.7 mm
- net N$48: track 17.3 -> 20.1 mm
- net N$39: track 17.3 -> 20.1 mm
- net N$61: track 22.7 -> 25.4 mm
- net N$38: track 16.8 -> 19.4 mm
- net N$40: track 17.8 -> 20.4 mm
- net N$34: track 20.4 -> 22.9 mm
- net N$43: track 20.3 -> 22.6 mm
- net N$46: track 16.8 -> 19.1 mm
- net N$45: track 17.8 -> 20.2 mm
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Other:
- board text added: "A"
- board text added: "AC15V/1A"
- board text added: "B"
- board text removed: "AC24V"
