File: snowmaker/SnowMaker_V1.0.sch (EAGLE design)
At the start: 570 parts, among them CON1 HR951180A, CON2 SWJ, IC1 ST3232BD, IC10 LM1117IDTX-3.3, IC11 SGM8584XS14, IC12 LM78M24, IC13 SGM8584XS14, IC14 SGM8584XS14, IC15 SGM8584XS14, IC2 ST3485EBD, IC3 W5500, IC4 SD2068, IC5 STM32F103VCT6, IC6 ULN2803, IC7 ULN2803, IC8 ULN2803, IC9 LM4040AIM3X-2.5, U1 LQ-BTM2540, X10 FFKDS/V1-5.08_MIDDLE, X11 FFKDS/V1-5.08_MIDDLE, X12 FFKDS/V1-5.08_MIDDLE, X13 FFKDS/V1-5.08_MIDDLE, X14 FFKDS/V1-5.08_MIDDLE, X15 FFKDS/V1-5.08_MIDDLE, X16 FFKDS/V1-5.08_MIDDLE, X17 FFKDS/V1-5.08_MIDDLE, X18 FFKDS/V1-5.08_MIDDLE, X19 FFKDS/V1-5.08_MIDDLE, X2 FFKDS/V1-5.08_FIRST, X20 FFKDS/V1-5.08_MIDDLE, X21 FFKDS/V1-5.08_MIDDLE, X22 FFKDS/V1-5.08_MIDDLE, X23 FFKDS/V1-5.08_MIDDLE, X24 FFKDS/V1-5.08_MIDDLE, X25 FFKDS/V1-5.08_MIDDLE, X26 FFKDS/V1-5.08_MIDDLE, X27 FFKDS/V1-5.08_MIDDLE, X28 FFKDS/V1-5.08_MIDDLE, X29 FFKDS/V1-5.08_MIDDLE, X3 FFKDS/V1-5.08_MIDDLE, X30 FFKDS/V1-5.08_MIDDLE, X31 FFKDS/V1-5.08_MIDDLE, X32 FFKDS/V1-5.08_MIDDLE, X33 FFKDS/V1-5.08_MIDDLE, X34 FFKDS/V1-5.08_MIDDLE, X35 FFKDS/V1-5.08_MIDDLE, X36 FFKDS/V1-5.08_MIDDLE, X37 FFKDS/V1-5.08_MIDDLE, X38 FFKDS/V1-5.08_MIDDLE, X39 FFKDS/V1-5.08_MIDDLE, X4 FFKDS/V1-5.08_MIDDLE, X40 FFKDS/V1-5.08_MIDDLE, X41 FFKDS/V1-5.08_LAST, X42 FFKDS/V1-5.08_MIDDLE, X43 FFKDS/V1-5.08_LAST, X44 FFKDS/V1-5.08_MIDDLE, X45 FFKDS/V1-5.08_MIDDLE, X46 FFKDS/V1-5.08_MIDDLE, X47 FFKDS/V1-5.08_MIDDLE, X48 FFKDS/V1-5.08_MIDDLE, X49 FFKDS/V1-5.08_MIDDLE, X5 FFKDS/V1-5.08_MIDDLE, X50 FFKDS/V1-5.08_MIDDLE, X51 FFKDS/V1-5.08_MIDDLE, X52 FFKDS/V1-5.08_MIDDLE, X53 FFKDS/V1-5.08_MIDDLE, X54 FFKDS/V1-5.08_MIDDLE, X55 FFKDS/V1-5.08_MIDDLE, X56 FFKDS/V1-5.08_MIDDLE, X57 FFKDS/V1-5.08_MIDDLE, X58 FFKDS/V1-5.08_FIRST, X59 FFKDS/V1-5.08_MIDDLE, X6 FFKDS/V1-5.08_MIDDLE, X60 FFKDS/V1-5.08_MIDDLE, X61 FFKDS/V1-5.08_MIDDLE, X62 FFKDS/V1-5.08_MIDDLE, X63 FFKDS/V1-5.08_MIDDLE, X64 FFKDS/V1-5.08_MIDDLE, X65 FFKDS/V1-5.08_MIDDLE, X66 FFKDS/V1-5.08_MIDDLE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

Commit message: PI fisrt commit
Connections:
- net N$61: now also X1.8
- net N$62: now also X1.6, X1.7; no longer X1.8
Other:
- note added: "XT1 15VAC/1A Power Supply"
- note added: "至迪文触摸屏 低温，两个版本（-30、-40） 需要对端板做供电，无需做电平转换。"
- note removed: "6-24V DC/DC Power Supply"
- note removed: "至迪文触摸屏 低温，两个版本（-30、-40） 需要对端做供电以及电平转换板。"
- moved on the sheet: C10, C11, C12, C2, C3, C7, C9, F3, IC1, L1, R1, R12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
