File: PannelInterface/PannelInterface.brd (EAGLE design)
At the start: 45 x 100 mm, 10 parts, among them IC2 LM2575D2T-012

Commit message: PI change
Parts:
- removed D1: SMDJ30A, SHMT:SMC
- added CON1: PH-8AW, prj-pannel_interface:PH-8AW
- added CON2: XH-8AW, prj-pannel_interface:XH-8AW
- added DB1: DB207S, prj-pannel_interface:DBS
- added LOGO1: SY-LOGO_BOTTOM, LOGO:SY-LOGO_BOTTOM
- C2: device rcl:UD-8X10_NICHICON -> rcl:TT5D11
- L1: value 330uH/2A_RH125 -> 330uH/2A_RH127
- moved C1 33.3 mm to (13.1, 35.8)
- moved C2 33.1 mm to (6.70, 30.8)
- moved D8 24.3 mm to (10.5, 51.7)
- moved L1 17.1 mm to (10.5, 60.0), turned to 90 degrees
- moved IC2 14.7 mm to (10.5, 43.5), turned to 90 degrees
- moved C3 13.4 mm to (11.5, 71.4), turned to 0 degrees
- moved C9 9.16 mm to (11.5, 77.7)
- moved X1 8.99 mm to (24.5, 31.5)
Connections:
- new net AC1: DB1.AC2, X1.6, X1.7
- new net AC2: DB1.AC1, X1.8, X1.9
- new net RXD: CON1.6, CON2.5, CON2.6, X1.2
- new net TXD: CON1.5, CON2.4, X1.3
- net +12V: now also CON1.1, CON1.2, CON2.1, CON2.2
- net GND: now also CON1.7, CON1.8, CON2.7, CON2.8, DB1.-, X1.G1, X1.G2; no longer D1.A
- net N$1: now also DB1.+; no longer D1.C
Routing:
- net +12V: track 0.00 -> 97.3 mm
- net AC1: track 0.00 -> 72.6 mm
- net RXD: track 0.00 -> 72.3 mm
- net TXD: track 0.00 -> 68.9 mm
- net AC2: track 0.00 -> 58.8 mm
- net N$34: track 0.00 -> 41.0 mm, vias 0 -> 2
- net GND: track 0.00 -> 28.8 mm, vias 0 -> 22
- net N$1: track 0.00 -> 20.9 mm
- added copper zone on layer 1, net GND
- added copper zone on layer 16, net GND
- added copper zone on layer 1, net N$34
Other:
- board size 45 x 100 mm -> 36 x 100 mm
- board text added: "SMTLCMIB-V1.0"

Commit message: update
Parts:
- removed C9: 100n/50V, SHMT:C0805
- removed D8: SS14, SHMT:SMA-DO214AC
- added C4: 100n/50V, SHMT:C0805
- added D1: SS24, SHMT:DO214AA
- C3: value 330uF/10V -> 330uF/16V
- CON1: value PH-8AW -> XH-8AW; device prj-pannel_interface:PH-8AW -> prj-pannel_interface:XH-8AW
- CON2: value XH-8AW -> PH-8AW; device prj-pannel_interface:XH-8AW -> prj-pannel_interface:PH-8AW
- moved CON1 26.8 mm to (26.7, 53.2)
- moved CON2 26.8 mm to (29.6, 79.9)
- moved L1 0.92 mm to (10.3, 60.8)
- moved C3 0.51 mm to (11.5, 71.9)
- renumbered IC2 to IC1
Connections:
- net +12V: now also C4.1; no longer C9.1
- net GND: now also C4.2, D1.A; no longer C9.2, D8.A
- net N$34: now also D1.C; no longer D8.C
- net RXD: now also CON1.5; no longer CON2.5
- net TXD: now also CON1.4, CON2.5; no longer CON1.5, CON2.4
Routing:
- net +12V: track 97.3 -> 52.4 mm
- net N$34: track 41.0 -> 0.00 mm, vias 2 -> 5
- net N$1: track 20.9 -> 7.44 mm
- net GND: track 28.8 -> 21.3 mm, vias 22 -> 88
- net AC2: track 58.8 -> 63.0 mm
- net RXD: track 72.3 -> 69.0 mm
- net AC1: track 72.6 -> 75.2 mm
- added copper zone on layer 1, net +12V
- added copper zone on layer 1, net N$1
- added copper zone on layer 16, net N$34
