File: PannelInterface/PannelInterface.sch (EAGLE design)
At the start: 12 parts, among them CON1 PH-8AW, CON2 XH-8AW, IC2 LM2575D2T-012

Commit message: update
Parts:
- removed D8: SS14, SHMT:SCHOTTKY-DIODE
- added D1: SS24, SHMT:SCHOTTKY-DIODE-SS24
- C3: value 330uF/10V -> 330uF/16V
- CON1: value PH-8AW -> XH-8AW; device prj-pannel_interface:PH-8AW -> prj-pannel_interface:XH-8AW
- CON2: value XH-8AW -> PH-8AW; device prj-pannel_interface:XH-8AW -> prj-pannel_interface:PH-8AW
- renumbered C9 to C4, IC2 to IC1
Connections:
- net GND: now also D1.A; no longer D8.A
- net N$34: now also D1.C; no longer D8.C
- net RXD: now also CON1.5; no longer CON2.5
- net TXD: now also CON1.4, CON2.5; no longer CON1.5, CON2.4
Other:
- note added: "触摸屏转接适配板"
- moved on the sheet: CON1, CON2
