File: DevTool/devtool.brd (EAGLE design)
At the start: 100 x 80 mm, 28 parts, among them IC1 SGM8584XS14, IC2 SGM8584XS14, IC3 SGM8584XS14, IC4 7805T

Commit message: continue
Parts:
- added C1, C10, C11, C12, C13, C14, C15, C16, C17, C2, C3, C4, C5, C6, C7, C8, C9: 100nF/50V, SHMT:C0603
- added IC5: TL431, SHMT:SOT23-3
- added R13, R14, R15, R16, R17, R18, R19, R20, R21, R22, R23, R24, R25: 10K, SHMT:R0603
- added RP1, RP10, RP11, RP12, RP2, RP3, RP4, RP5, RP6, RP7, RP8, RP9: 20K, SHMT:RM065
- added SW1, SW10, SW11, SW12, SW13, SW14, SW15, SW16, SW17, SW18, SW19, SW2, SW20, SW3, SW4, SW5, SW6, SW7, SW8, SW9: PB-22E60, SHMT:PB-22E60
- moved Q10 81.8 mm to (-24.1, 61.0)
- moved Q11 81.8 mm to (-29.2, 53.3)
- moved Q12 81.8 mm to (-24.1, 53.3)
- moved Q2 81.8 mm to (-14.0, 85.1)
- moved Q3 81.8 mm to (-21.6, 85.1)
- moved Q4 81.8 mm to (-29.2, 85.1)
- moved Q5 81.8 mm to (-29.2, 76.2)
- moved Q6 81.8 mm to (-24.1, 76.2)
- moved Q7 81.8 mm to (-29.2, 68.6)
- moved Q8 81.8 mm to (-24.1, 68.6)
- moved Q9 81.8 mm to (-29.2, 61.0)
- moved R1 81.8 mm to (-29.2, 47.0)
- moved R10 81.8 mm to (-29.2, 1.27)
- moved R11 81.8 mm to (-29.2, -3.81)
- moved R12 81.8 mm to (-29.2, -8.89)
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Connections:
- new net +24V: C17.1, IC4.1, SW1.2, SW1.5, SW10.2, SW10.5, SW11.2, SW11.5, SW12.2, SW12.5, SW13.2, SW14.2, SW14.5, SW15.2, SW15.5, SW16.2, SW16.3, SW16.6, SW17.2, SW17.5, SW18.2, SW18.5, SW19.2, SW19.5, SW2.2, SW2.5, SW20.2, SW20.5, SW3.2, SW3.5, SW4.2, SW4.5, SW5.2, SW6.2, SW7.2, SW8.2, SW8.3, SW8.5, SW8.6, SW9.2, SW9.5
- new net N$1: SW12.3, SW12.6
- new net N$26: SW14.3, SW14.6
- new net N$27: SW14.1, SW14.4
- new net N$28: SW13.1, SW13.4
- new net N$29: SW15.1, SW15.4
- new net N$30: SW15.3, SW15.6
- new net N$31: SW16.1, SW16.4
- new net N$32: SW8.1, SW8.4
- new net N$33: SW7.3, SW7.6
- new net N$34: SW7.1, SW7.4
- new net N$35: SW6.3, SW6.6
- new net N$36: SW6.1, SW6.4
- new net N$37: SW5.3, SW5.6
- new net N$38: SW5.1, SW5.4
- new net N$39: SW4.3, SW4.6
- new net N$40: SW4.1, SW4.4
- new net N$41: SW3.1, SW3.4
- new net N$42: SW3.3, SW3.6
- new net N$43: SW2.1, SW2.4
- new net N$44: SW2.3, SW2.6
- new net N$45: SW1.3, SW1.6
- new net N$46: SW1.1, SW1.4
- new net N$47: SW9.1, SW9.4
- new net N$48: SW9.3, SW9.6
- new net N$49: SW10.1, SW10.4
- new net N$50: SW10.3, SW10.6
- new net N$51: SW11.1, SW11.4
- new net N$52: SW11.3, SW11.6
- new net N$53: SW12.1, SW12.4
- new net N$54: C1.1, R13.1, RP1.3
- new net N$55: C2.1, R14.1, RP2.3
- new net N$56: C3.1, R15.1, RP3.3
- new net N$57: C4.1, R16.1, RP4.3
- new net N$58: C5.1, R17.1, RP5.3
- new net N$59: C6.1, R18.1, RP6.3
- new net N$60: C7.1, R19.1, RP7.3
- new net N$61: C8.1, R20.1, RP8.3
- new net N$62: C9.1, R21.1, RP9.3
- new net N$63: C10.1, R22.1, RP10.3
- new net N$64: C11.1, R23.1, RP11.3
- new net N$65: C12.1, R24.1, RP12.3
- new net N$66: IC1.3, R13.2
- new net N$67: IC1.5, R14.2
- new net N$68: IC1.10, R15.2
- new net N$69: IC1.12, R16.2
- new net N$70: IC2.12, R20.2
- new net N$71: IC2.10, R19.2
- new net N$72: IC2.5, R18.2
- new net N$73: IC2.3, R17.2
- new net N$74: IC3.3, R21.2
- new net N$75: IC3.5, R22.2
- new net N$76: IC3.10, R23.2
- new net N$77: IC3.12, R24.2
- new net REF: IC5.1, IC5.2, R25.1, RP1.2, RP10.2, RP11.2, RP12.2, RP2.2, RP3.2, RP4.2, RP5.2, RP6.2, RP7.2, RP8.2, RP9.2
- net +5V: now also C13.1, C14.1, C15.1, C16.1, R25.2
- net GND: now also C1.2, C10.2, C11.2, C12.2, C13.2, C14.2, C15.2, C16.2, C17.2, C2.2, C3.2, C4.2, C5.2, C6.2, C7.2, C8.2, C9.2, IC5.3, RP1.1, RP10.1, RP11.1, RP12.1, RP2.1, RP3.1, RP4.1, RP5.1, RP6.1, RP7.1, RP8.1, RP9.1
